Commit message: 實體可以正常控制，但是有一個問題手臂移動會不准，下一個版本修復

File: src/ar4_hardware_interface/urdf/ar4.ros2_control_hardware.xacro (robot description, xacro)
@@ -8,4 +8,20 @@
     joint_offset_parameters_file
   ">
+      <!-- 定義角度轉弧度常數 -->
+    <xacro:property name="deg_to_rad" value="${pi / 180}" />
+    <!-- 各關節的 position limits（單位：弧度） -->
+    <xacro:property name="j1_min" value="${-170 * deg_to_rad}" />
+    <xacro:property name="j1_max" value="${ 170 * deg_to_rad}" />
+    <xacro:property name="j2_min" value="${-42 * deg_to_rad}" />
+    <xacro:property name="j2_max" value="${ 90 * deg_to_rad}" />
+    <xacro:property name="j3_min" value="${-89 * deg_to_rad}" />
+    <xacro:property name="j3_max" value="${ 52 * deg_to_rad}" />
+    <xacro:property name="j4_min" value="${-165 * deg_to_rad}" />
+    <xacro:property name="j4_max" value="${ 165 * deg_to_rad}" />
+    <xacro:property name="j5_min" value="${-105 * deg_to_rad}" />
+    <xacro:property name="j5_max" value="${ 105 * deg_to_rad}" />
+    <xacro:property name="j6_min" value="${-155 * deg_to_rad}" />
+    <xacro:property name="j6_max" value="${ 155 * deg_to_rad}" />
+    <!-- ====================================================== -->
     <xacro:property name="joint_offset_parameters"
       value="${xacro.load_yaml(joint_offset_parameters_file)}"/>
@@ -18,6 +34,6 @@
       <joint name="joint_1">
         <command_interface name="position">
-          <param name="min">{-170*pi/180}</param>
-          <param name="max">{170*pi/180}</param>
+          <param name="min">${j1_min}</param>
+          <param name="max">${j1_max}</param>
         </command_interface>
         <state_interface name="position">
@@ -28,6 +44,6 @@
       <joint name="joint_2">
         <command_interface name="position">
-          <param name="min">{-42*pi/180}</param>
-          <param name="max">{90*pi/180}</param>
+          <param name="min">${j2_min}</param>
+          <param name="max">${j2_max}</param>
         </command_interface>
         <state_interface name="position">
@@ -38,6 +54,6 @@
       <joint name="joint_3">
         <command_interface name="position">
-          <param name="min">{-89*pi/180}</param>
-          <param name="max">{52*pi/180}</param>
+          <param name="min">${j3_min}</param>
+          <param name="max">${j3_max}</param>
         </command_interface>
         <state_interface name="position">
@@ -48,6 +64,6 @@
       <joint name="joint_4">
         <command_interface name="position">
-          <param name="min">{-165*pi/180}</param>
-          <param name="max">{165*pi/180}</param>
+          <param name="min">${j4_min}</param>
+          <param name="max">${j4_max}</param>
         </command_interface>
         <state_interface name="position">
@@ -58,6 +74,6 @@
       <joint name="joint_5">
         <command_interface name="position">
-          <param name="min">{-105*pi/180}</param>
-          <param name="max">{105*pi/180}</param>
+          <param name="min">${j5_min}</param>
+          <param name="max">${j5_max}</param>
         </command_interface>
         <state_interface name="position">
@@ -68,6 +84,6 @@
       <joint name="joint_6">
         <command_interface name="position">
-          <param name="min">{-155*pi/180}</param>
-          <param name="max">{155*pi/180}</param>
+          <param name="min">${j6_min}</param>
+          <param name="max">${j6_max}</param>
         </command_interface>
         <state_interface name="position">

File: src/ar4_hardware_interface/urdf/ar4.urdf.xacro (robot description, xacro)
@@ -8,6 +8,7 @@
   <xacro:include filename="$(find ar4_description)/urdf/ar4.urdf.xacro"/>
   <xacro:include filename="$(find ar4_hardware_interface)/urdf/ar4.ros2_control_hardware.xacro"/>
+  <xacro:include filename="$(find ar4_hardware_interface)/urdf/ar4_gripper.ros2_control_hardware.xacro"/>
   <link name="world" />
-  <joint name="base_joint" type="fixed">
+  <joint name="joint_world" type="fixed">
     <origin xyz="0 0 0" rpy="0 0 0" />
       <parent link="world"/>
@@ -21,3 +22,10 @@
     joint_offset_parameters_file="$(find ar4_hardware_interface)/config/joint_offsets/ar4.yaml"
   />
+  <xacro:ar_gripper_ros2_control
+    name="ar4_gripper"
+    plugin_name="ar4_hardware_interface/ARSwitchGripperHWInterface"
+    serial_port="$(arg arduino_serial_port)"
+    calibrate="$(arg calibrate)"
+    joint_offset_parameters_file="$(find ar4_hardware_interface)/config/joint_offsets/ar4.yaml"
+  />
 </robot>

File: src/ar4_moveit_config/config/ar4.ros2_control.xacro (robot description, xacro)
@@ -6,5 +6,5 @@
             <hardware>
                 <!-- By default, set up controllers for simulation. This won't work on real hardware -->
-                <plugin>gz_ros2_control/GazeboSimSystem</plugin>
+                <plugin>mock_components/GenericSystem</plugin>
             </hardware>
             <joint name="joint_1">
@@ -13,5 +13,4 @@
                   <param name="initial_value">${initial_positions['joint_1']}</param>
                 </state_interface>
-                <state_interface name="velocity"/>
             </joint>
             <joint name="joint_2">
@@ -20,5 +19,4 @@
                   <param name="initial_value">${initial_positions['joint_2']}</param>
                 </state_interface>
-                <state_interface name="velocity"/>
             </joint>
             <joint name="joint_3">
@@ -27,5 +25,4 @@
                   <param name="initial_value">${initial_positions['joint_3']}</param>
                 </state_interface>
-                <state_interface name="velocity"/>
             </joint>
             <joint name="joint_4">
@@ -34,5 +31,4 @@
                   <param name="initial_value">${initial_positions['joint_4']}</param>
                 </state_interface>
-                <state_interface name="velocity"/>
             </joint>
             <joint name="joint_5">
@@ -41,5 +37,4 @@
                   <param name="initial_value">${initial_positions['joint_5']}</param>
                 </state_interface>
-                <state_interface name="velocity"/>
             </joint>
             <joint name="joint_6">
@@ -48,5 +43,4 @@
                   <param name="initial_value">${initial_positions['joint_6']}</param>
                 </state_interface>
-                <state_interface name="velocity"/>
             </joint>
             <joint name="grip_to_base1">
@@ -55,5 +49,4 @@
                   <param name="initial_value">${initial_positions['grip_to_base1']}</param>
                 </state_interface>
-                <state_interface name="velocity"/>
             </joint>
         </ros2_control>

File: src/ar4_moveit_config/config/ar4.urdf.xacro (robot description, xacro)
@@ -3,7 +3,7 @@
     <xacro:arg name="initial_positions_file" default="initial_positions.yaml" />
     <!-- Import ar4 urdf file -->
-    <xacro:include filename="$(find ar4_description)/urdf/ar4_in_world.urdf.xacro" />
+    <xacro:include filename="$(find ar4_description)/urdf/ar4.urdf.xacro" />
     <!-- Import control_xacro -->
     <xacro:include filename="ar4.ros2_control.xacro" />
-    <xacro:ar4_ros2_control name="ar4" initial_positions_file="$(arg initial_positions_file)"/>
+    <xacro:ar4_ros2_control name="FakeSystem" initial_positions_file="$(arg initial_positions_file)"/>
 </robot>
