Commit message: 模擬夾爪可以同步打開，實體手臂問題在下一個版本解決

File: src/ar4_gazebo_sim/urdf/includes/ar4.ros2_control.xacro (robot description, xacro)
@@ -57,4 +57,12 @@
                 <state_interface name="velocity"/>
             </joint>
+            <joint name="grip_to_base2">
+                <param name="mimic">grip_to_base1</param>
+                <param name="multiplier">1</param>
+            </joint>
+            <joint name="grip_to_base3">
+                <param name="mimic">grip_to_base1</param>
+                <param name="multiplier">1</param>
+            </joint>
         </ros2_control>
     </xacro:macro>
