Commit message: 新增深度相機裝到手臂末端，模擬的深度相機有功能，實體的還沒有

File: src/ar4_description/urdf/ar4.urdf.xacro (robot description, xacro)
@@ -111,13 +111,46 @@
     <child link="cylinder"/>
   </joint>
+  <!-- Link cylinder -->
   <link name="cylinder">
     <inertial>
       <origin xyz="0 0 0" rpy="0 0 0"/>
-      <mass value="0.1"/>
-      <inertia ixx="0.001" ixy="0" ixz="0" iyy="0.001" iyz="0" izz="0.001"/>
-    </inertial>
+      <mass value="0.01"/>
+      <inertia ixx="0.0001" ixy="0" ixz="0" iyy="0.0001" iyz="0" izz="0.0001"/>
+    </inertial>
+    <!-- Part arm_holder -->
+    <visual>
+      <origin xyz="0 0 0.006" rpy="1.5708 0 -3.14159"/>
+      <geometry>
+        <mesh filename="file://$(find ar4_description)/meshes//arm_holder.stl"/>
+      </geometry>
+      <material name="arm_holder_material">
+        <color rgba="0.980392 0.713725 0.00392157 1"/>
+      </material>
+    </visual>
+    <collision>
+      <origin xyz="0 0 0.006" rpy="1.5708 0 -3.14159"/>
+      <geometry>
+        <mesh filename="file://$(find ar4_description)/meshes/arm_holder.stl"/>
+      </geometry>
+    </collision>
+    <!-- Part deep_camera -->
+    <visual>
+      <origin xyz="0 0.08157 0.039" rpy="-0 0 -3.14159"/>
+      <geometry>
+        <mesh filename="file://$(find ar4_description)/meshes/deep_camera.stl"/>
+      </geometry>
+      <material name="deep_camera_material">
+        <color rgba="1 1 1 1"/>
+      </material>
+    </visual>
+    <collision>
+      <origin xyz="0 0.08157 0.039" rpy="-0 0 -3.14159"/>
+      <geometry>
+        <mesh filename="file://$(find ar4_description)/meshes/deep_camera.stl"/>
+      </geometry>
+    </collision>
     <!-- Part cylinder -->
     <visual>
-      <origin xyz="0 0 0" rpy="1.5708 -0 -0"/>
+      <origin xyz="0 0 0.006" rpy="1.5708 -0 -3.14159"/>
       <geometry>
         <mesh filename="file://$(find ar4_description)/meshes/cylinder.stl"/>
@@ -128,29 +161,75 @@
     </visual>
     <collision>
-      <origin xyz="0 0 0" rpy="1.5708 -0 -0"/>
+      <origin xyz="0 0 0.006" rpy="1.5708 -0 -3.14159"/>
       <geometry>
         <mesh filename="file://$(find ar4_description)/meshes/cylinder.stl"/>
       </geometry>
     </collision>
-  </link>
+    <!-- Part deep_camera_holder -->
+    <visual>
+      <origin xyz="0 -0.0003 0.006" rpy="-1.5708 0 -3.14159"/>
+      <geometry>
+        <mesh filename="file://$(find ar4_description)/meshes/deep_camera_holder.stl"/>
+      </geometry>
+      <material name="deep_camera_holder_material">
+        <color rgba="0.980392 0.713725 0.00392157 1"/>
+      </material>
+    </visual>
+    <collision>
+      <origin xyz="0 -0.0003 0.006" rpy="-1.5708 0 -3.14159"/>
+      <geometry>
+        <mesh filename="file://$(find ar4_description)/meshes/deep_camera_holder.stl"/>
+      </geometry>
+    </collision>
+  </link>
+  <!-- Frame camera (dummy link + fixed joint) -->
+  <link name="camera">
+    <origin xyz="0 0 0" rpy="0 -0 0"/>
+    <inertial>
+      <origin xyz="0 0 0" rpy="0 0 0"/>
+      <mass value="0.01"/>
+      <inertia ixx="0.0001" ixy="0" ixz="0" iyy="0.0001" iyz="0" izz="0.0001"/>
+    </inertial>
+  </link>
+  <joint name="camera_frame" type="fixed">
+    <origin xyz="0.0301 0.08157 0.036" rpy="-0 0 -3.14159"/>
+    <parent link="cylinder"/>
+    <child link="camera"/>
+    <axis xyz="0 0 0"/>
+  </joint>
+  <!-- Frame depth_camera (dummy link + fixed joint) -->
+  <link name="depth_camera">
+    <origin xyz="0 0 0" rpy="0 -0 0"/>
+    <inertial>
+      <origin xyz="0 0 0" rpy="0 0 0"/>
+      <mass value="0.01"/>
+      <inertia ixx="0.0001" ixy="0" ixz="0" iyy="0.0001" iyz="0" izz="0.0001"/>
+    </inertial>
+  </link>
+  <joint name="depth_camera_frame" type="fixed">
+    <origin xyz="-0.0019 0.08157 0.036" rpy="1.570795 -1.570795 -3.14159"/>
+    <parent link="cylinder"/>
+    <child link="depth_camera"/>
+    <axis xyz="0 0 0"/>
+  </joint>
   <!-- Link gripper -->
   <link name="gripper">
     <inertial>
       <origin xyz="0 0 0" rpy="0 0 0"/>
-      <mass value="0.1"/>
+      <mass value="0.01"/>
       <inertia ixx="0.001" ixy="0" ixz="0" iyy="0.001" iyz="0" izz="0.001"/>
     </inertial>
     <!-- Part gripper -->
     <visual>
-      <origin xyz="-0.056 0.0249 0.003" rpy="1.5708 1.5708 0"/>
+      <origin xyz="-0.0495 -0.0249 0.003" rpy="-1.5708 -1.5708 0"/>
       <geometry>
         <mesh filename="file://$(find ar4_description)/meshes/gripper.stl"/>
       </geometry>
       <material name="gripper_material">
-        <color rgba="0.647059 0.647059 0.647059 1"/>
-      </material>
-    </visual>
-    <collision>
-      <origin xyz="-0.056 0.0249 0.003" rpy="1.5708 1.5708 0"/>
+        <color rgba="0.980392 0.713725 0.00392157 1"/>
+      </material>
+    </visual>
+    <collision>
+      <origin xyz="-0.0495 -0.0249 0.003" rpy="-1.5708 -1.5708 0"/>
       <geometry>
         <mesh filename="file://$(find ar4_description)/meshes/gripper.stl"/>
@@ -160,9 +239,9 @@
   <!-- Joint from cylinder to gripper -->
   <joint name="grip_to_base1" type="revolute">
-    <origin xyz="0.003 -0.0249 0.056" rpy="-1.5708 -1.26477 1.5708"/>
+    <origin xyz="0.020064 -0.0150481 0.0545" rpy="1.5708 -1.0821 2.61799"/>
     <parent link="cylinder"/>
     <child link="gripper"/>
     <axis xyz="0 0 1"/>
-    <limit effort="10" velocity="10" lower="-0.916889" upper="0.182668"/>
+    <limit effort="10" velocity="10" lower="-0.001" upper="0.488692"/>
   </joint>
   <!-- Link gripper_2 -->
@@ -170,19 +249,19 @@
     <inertial>
       <origin xyz="0 0 0" rpy="0 0 0"/>
-      <mass value="0.1"/>
+      <mass value="0.01"/>
       <inertia ixx="0.001" ixy="0" ixz="0" iyy="0.001" iyz="0" izz="0.001"/>
     </inertial>
     <!-- Part gripper_2 -->
     <visual>
-      <origin xyz="-0.056 -0.0249 0.003" rpy="-1.5708 -1.5708 0"/>
+      <origin xyz="-0.0495 -0.0249 0.003" rpy="-1.5708 -1.5708 0"/>
       <geometry>
         <mesh filename="file://$(find ar4_description)/meshes/gripper.stl"/>
       </geometry>
       <material name="gripper_2_material">
-        <color rgba="0.647059 0.647059 0.647059 1"/>
-      </material>
-    </visual>
-    <collision>
-      <origin xyz="-0.056 -0.0249 0.003" rpy="-1.5708 -1.5708 0"/>
+        <color rgba="0.980392 0.713725 0.00392157 1"/>
+      </material>
+    </visual>
+    <collision>
+      <origin xyz="-0.0495 -0.0249 0.003" rpy="-1.5708 -1.5708 0"/>
       <geometry>
         <mesh filename="file://$(find ar4_description)/meshes/gripper.stl"/>
@@ -192,10 +271,10 @@
   <!-- Joint from cylinder to gripper_2 -->
   <joint name="grip_to_base2" type="revolute">
-    <origin xyz="-0.020064 0.0150481 0.056" rpy="1.5708 -1.26477 -0.523599"/>
+    <origin xyz="-0.023064 -0.00985192 0.0545" rpy="1.5708 -1.0821 0.523599"/>
     <parent link="cylinder"/>
     <child link="gripper_2"/>
     <axis xyz="0 0 1"/>
-    <limit effort="10" velocity="10" lower="-0.182668" upper="0.916889"/>
-    <mimic joint="grip_to_base1" multiplier="-1.0"/>
+    <limit effort="10" velocity="10" lower="-0.001" upper="0.488692"/>
+    <mimic joint="grip_to_base1" multiplier="1.0"/>
   </joint>
   <!-- Link gripper_3 -->
@@ -203,19 +282,19 @@
     <inertial>
       <origin xyz="0 0 0" rpy="0 0 0"/>
-      <mass value="0.1"/>
+      <mass value="0.01"/>
       <inertia ixx="0.001" ixy="0" ixz="0" iyy="0.001" iyz="0" izz="0.001"/>
     </inertial>
     <!-- Part gripper_3 -->
     <visual>
-      <origin xyz="-0.056 0.0249 0.003" rpy="1.5708 1.5708 0"/>
+      <origin xyz="-0.0495 -0.0249 0.003" rpy="-1.5708 -1.5708 0"/>
       <geometry>
         <mesh filename="file://$(find ar4_description)/meshes/gripper.stl"/>
       </geometry>
       <material name="gripper_3_material">
-        <color rgba="0.647059 0.647059 0.647059 1"/>
-      </material>
-    </visual>
-    <collision>
-      <origin xyz="-0.056 0.0249 0.003" rpy="1.5708 1.5708 0"/>
+        <color rgba="0.980392 0.713725 0.00392157 1"/>
+      </material>
+    </visual>
+    <collision>
+      <origin xyz="-0.0495 -0.0249 0.003" rpy="-1.5708 -1.5708 0"/>
       <geometry>
         <mesh filename="file://$(find ar4_description)/meshes/gripper.stl"/>
@@ -225,10 +304,10 @@
   <!-- Joint from cylinder to gripper_3 -->
   <joint name="grip_to_base3" type="revolute">
-    <origin xyz="0.020064 0.0150481 0.056" rpy="-1.5708 -1.26477 -2.61799"/>
+    <origin xyz="0.003 0.0249 0.0545" rpy="1.5708 -1.0821 -1.5708"/>
     <parent link="cylinder"/>
     <child link="gripper_3"/>
     <axis xyz="0 0 1"/>
-    <limit effort="10" velocity="10" lower="-0.916889" upper="0.182668"/>
-    <mimic joint="grip_to_base2" multiplier="-1.0"/>
+    <limit effort="10" velocity="10" lower="-0.001" upper="0.488692"/>
+    <mimic joint="grip_to_base1" multiplier="1.0"/>
   </joint>
 </robot>

File: src/ar4_description/urdf/ar4_in_world.urdf.xacro (robot description, xacro)
@@ -6,5 +6,6 @@
     <parent link="world" />
     <child link="base_link" />
-    <origin xyz="0 0 0" rpy="0 0 ${-pi/2}" />
+    <origin xyz="0 0 0" rpy="0 0 0" />
+    <!-- <origin xyz="0 0 0" rpy="0 0 ${-pi/2}" /> -->
   </joint>
 </robot>

File: src/ar4_gazebo_sim/urdf/includes/gazebo.xacro (robot description, xacro)
@@ -28,3 +28,24 @@
         </plugin>
     </gazebo>
+    <gazebo reference="depth_camera">
+      <sensor name="depth_camera" type="rgbd_camera">
+        <update_rate>30</update_rate>
+        <topic>depth_camera</topic>
+        <gz_frame_id>depth_camera</gz_frame_id>
+        <always_on>true</always_on>
+        <visualize>true</visualize>
+        <camera>
+          <horizontal_fov>1.047</horizontal_fov>
+          <image>
+            <width>640</width>
+            <height>480</height>
+            <format>R8G8B8</format>
+          </image>
+          <clip>
+            <near>0.05</near>
+            <far>10.0</far>
+          </clip>
+        </camera>
+      </sensor>
+    </gazebo>
 </robot>

Commit message: 可以找到架子的點，然後寫一些手臂一到未來的程式，但未完成，並且流程已經寫好，還有加一些測試程式

File: src/ar4_description/urdf/ar4.urdf.xacro (robot description, xacro)
@@ -311,3 +311,11 @@
     <mimic joint="grip_to_base1" multiplier="1.0"/>
   </joint>
+  <!-- Frame gripper_tcp (Tool Center Point) -->
+  <link name="gripper_tcp"/>
+  <joint name="gripper_tcp_joint" type="fixed">
+    <!-- 這裡的 xyz 可以根據您夾爪末端的實際距離進行微調，目前 z 暫設為 0.1515 (15.15公分) -->
+    <origin xyz="0 0 0.1515" rpy="0 0 0"/>
+    <parent link="link_6"/>
+    <child link="gripper_tcp"/>
+  </joint>
 </robot>

File: src/ar4_gazebo_sim/urdf/includes/gazebo.xacro (robot description, xacro)
@@ -38,6 +38,6 @@
           <horizontal_fov>1.047</horizontal_fov>
           <image>
-            <width>640</width>
-            <height>480</height>
+            <width>1280</width>
+            <height>960</height>
             <format>R8G8B8</format>
           </image>

Commit message: 架子偵測方式改成yolo，將兩個service組合在一起，並增加去架子拿輪胎的程式，但是還未測試，底層驅動有改的比較不容易崩潰

File: src/ar4_description/urdf/ar4.urdf.xacro (robot description, xacro)
@@ -122,5 +122,5 @@
       <origin xyz="0 0 0.006" rpy="1.5708 0 -3.14159"/>
       <geometry>
-        <mesh filename="file://$(find ar4_description)/meshes//arm_holder.stl"/>
+        <mesh filename="file://$(find ar4_description)/meshes/arm_holder.stl"/>
       </geometry>
       <material name="arm_holder_material">
@@ -136,5 +136,5 @@
     <!-- Part deep_camera -->
     <visual>
-      <origin xyz="0 0.08157 0.039" rpy="-0 0 -3.14159"/>
+      <origin xyz="0 0.08157 0.039" rpy="-0 0 0"/>
       <geometry>
         <mesh filename="file://$(find ar4_description)/meshes/deep_camera.stl"/>
@@ -145,5 +145,5 @@
     </visual>
     <collision>
-      <origin xyz="0 0.08157 0.039" rpy="-0 0 -3.14159"/>
+      <origin xyz="0 0.08157 0.039" rpy="-0 0 0"/>
       <geometry>
         <mesh filename="file://$(find ar4_description)/meshes/deep_camera.stl"/>
@@ -193,9 +193,19 @@
   </link>
   <joint name="camera_frame" type="fixed">
-    <origin xyz="0.0301 0.08157 0.036" rpy="-0 0 -3.14159"/>
+    <origin xyz="-0.0301 0.08157 0.036" rpy="-0 0 0"/>
     <parent link="cylinder"/>
     <child link="camera"/>
     <axis xyz="0 0 0"/>
   </joint>
+  <link name="camera_color_optical_frame">
+    <origin xyz="0 0 0" rpy="0 -0 0"/>
+  </link>
+  <joint name="real_camera_frame" type="fixed">
+    <origin xyz="-0.0301 0.08157 0.036" rpy="1.570795 -1.570795 -3.14159"/>
+    <parent link="cylinder"/>
+    <child link="camera_color_optical_frame"/>
+    <axis xyz="0 0 0"/>
+  </joint>
+  <!-- Frame camera_depth_optical_frame (dummy link + fixed joint) -->
   <!-- Frame depth_camera (dummy link + fixed joint) -->
   <link name="depth_camera">
@@ -211,4 +221,13 @@
     <parent link="cylinder"/>
     <child link="depth_camera"/>
+    <axis xyz="0 0 0"/>
+  </joint>
+  <link name="camera_depth_optical_frame">
+    <origin xyz="0 0 0" rpy="0 -0 0"/>
+  </link>
+  <joint name="real_depth_camera_frame" type="fixed">
+    <origin xyz="-0.0019 0.08157 0.036" rpy="1.570795 -1.570795 -3.14159"/>
+    <parent link="cylinder"/>
+    <child link="camera_depth_optical_frame"/>
     <axis xyz="0 0 0"/>
   </joint>
@@ -312,8 +331,10 @@
   </joint>
   <!-- Frame gripper_tcp (Tool Center Point) -->
-  <link name="gripper_tcp"/>
+  <link name="gripper_tcp">
+    <origin xyz="0 0 0" rpy="0 -0 0"/>
+  </link>
   <joint name="gripper_tcp_joint" type="fixed">
     <!-- 這裡的 xyz 可以根據您夾爪末端的實際距離進行微調，目前 z 暫設為 0.1515 (15.15公分) -->
-    <origin xyz="0 0 0.1515" rpy="0 0 0"/>
+    <origin xyz="0 0 0.1566" rpy="0 0 0"/>
     <parent link="link_6"/>
     <child link="gripper_tcp"/>

File: src/ar4_gazebo_sim/urdf/includes/gazebo.xacro (robot description, xacro)
@@ -32,5 +32,6 @@
         <update_rate>60</update_rate>
         <topic>camera</topic>
-        <gz_frame_id>depth_camera</gz_frame_id>
+        <!-- <gz_frame_id>depth_camera</gz_frame_id> -->
+        <gz_frame_id>camera_color_optical_frame</gz_frame_id>
         <always_on>true</always_on>
         <visualize>true</visualize>
